File: bokstas_6_davikliai.kicad_pcb (KiCad board)
At the start: 2 copper layers, 42 parts, among them K7 OUT, Q1 BC817, Q2 BC817, U1 L7812, U2 4049, U3 NE555P

Commit message: versija 1.0
Parts:
- removed the D1 at (147.6, 67.9)
- removed the D2 at (163.8, 62.1)
- removed the D3 at (143.3, 71.2)
- removed the D4 at (153.9, 64.7)
- removed the D5 at (163.8, 55.6)
- removed the D6 at (149.7, 71.2)
- added C2: 100x35V, Capacitor_THT:CP_Radial_D8.0mm_P2.50mm, F.Cu at (166.0, 84.0)
- added C3: 330x16V, Capacitor_THT:CP_Radial_D8.0mm_P2.50mm, F.Cu at (130.8, 76.0)
- added D10: LL4007, Diode_SMD:D_MELF, B.Cu at (166.0, 89.0)
- added D7: BAS32, Diode_SMD:D_MiniMELF, B.Cu at (147.8, 76.8)
- added D8: LED, LED_THT:LED_D3.0mm, F.Cu at (160.2, 76.5)
- added J1: Sensors, Connector_PinHeader_2.54mm:PinHeader_1x10_P2.54mm_Vertical, F.Cu at (115.0, 83.1)
- added J2: LEDS, Connector_PinHeader_2.54mm:PinHeader_1x07_P2.54mm_Vertical, F.Cu at (146.1, 111.8)
- added J3: Conn_01x05, Connector_PinHeader_2.54mm:PinHeader_1x05_P2.54mm_Vertical, F.Cu at (166.0, 95.7)
- added R14: 10k, Resistor_THT:R_Axial_DIN0204_L3.6mm_D1.6mm_P7.62mm_Horizontal, F.Cu at (153.5, 93.2)
- added R15: 10k, Resistor_THT:R_Axial_DIN0204_L3.6mm_D1.6mm_P7.62mm_Horizontal, F.Cu at (153.5, 96.0)
- added R16: 10k, Resistor_THT:R_Axial_DIN0204_L3.6mm_D1.6mm_P7.62mm_Horizontal, F.Cu at (153.5, 98.5)
- added R17: 10k, Resistor_THT:R_Axial_DIN0204_L3.6mm_D1.6mm_P7.62mm_Horizontal, F.Cu at (153.5, 101.0)
- added R18: 10k, Resistor_THT:R_Axial_DIN0204_L3.6mm_D1.6mm_P7.62mm_Horizontal, F.Cu at (153.5, 103.5)
- added R19: 10k, Resistor_THT:R_Axial_DIN0204_L3.6mm_D1.6mm_P7.62mm_Horizontal, F.Cu at (153.5, 106.0)
- added R25: 10k, Resistor_SMD:R_0805_2012Metric, B.Cu at (157.2, 77.5)
- added REF**: MountingHole_2.1mm, MountingHole:MountingHole_2.1mm, F.Cu at (116.0, 112.0)
- added REF**: MountingHole_2.1mm, MountingHole:MountingHole_2.1mm, F.Cu at (116.0, 74.0)
- added REF**: MountingHole_2.1mm, MountingHole:MountingHole_2.1mm, F.Cu at (167.0, 74.0)
- added REF**: MountingHole_2.1mm, MountingHole:MountingHole_2.1mm, F.Cu at (167.0, 112.0)
- C4, C5, Q1, Q2, R10, R11, R12, R13, R8, R9: moved to B.Cu
- C6: value 47x25V -> 10x25V
- D1: renamed from D7; moved to B.Cu
- D2: renamed from D8; moved to B.Cu
- D3: renamed from D9; moved to B.Cu
- D4: renamed from D10; moved to B.Cu
- D5: renamed from D11; moved to B.Cu
- D6: renamed from D12; moved to B.Cu
- D9: renamed from D13; moved to B.Cu
- R1: footprint Resistor_SMD:R_0805_2012Metric -> Resistor_THT:R_Axial_DIN0204_L3.6mm_D1.6mm_P7.62mm_Horizontal
- R2, R3, R4, R5, R6, R7: value R -> 100k; footprint Resistor_SMD:R_0805_2012Metric -> Resistor_THT:R_Axial_DIN0204_L3.6mm_D1.6mm_P7.62mm_Horizontal
- R20: renamed from R14; moved to B.Cu
- R21: renamed from R15; moved to B.Cu
- R22: renamed from R16; moved to B.Cu
- R23: renamed from R17; value 100k -> 51k; moved to B.Cu
- R24: renamed from R18; moved to B.Cu
- U2: footprint Package_DIP:DIP-14_W7.62mm -> Package_DIP:DIP-16_W7.62mm
- moved R6 92.8 mm to (118.0, 103.5)
- moved R13 85.1 mm to (123.0, 106.0)
- moved R1 74.2 mm to (125.3, 88.2), turned to 180 degrees
- moved R7 73.5 mm to (118.0, 106.0)
- moved R2 71.7 mm to (118.0, 93.2)
- moved R10 68.8 mm to (123.0, 98.2)
- moved D5 68.6 mm to (149.7, 103.5), turned to 180 degrees
- moved R4 66.7 mm to (118.0, 98.2)
- moved R9 65.0 mm to (123.0, 95.8)
- moved D6 65.0 mm to (149.7, 106.0), turned to 180 degrees
- moved R12 63.5 mm to (123.0, 103.5)
- moved R3 58.4 mm to (118.0, 95.8)
- moved R8 58.3 mm to (123.0, 93.2)
- moved D1 56.6 mm to (149.7, 93.2), turned to 180 degrees
- moved R5 56.3 mm to (118.0, 101.0)
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- renumbered K7 to K1
Connections:
- D6 pad 2: Net-(D12-Pad2) -> Net-(D6-Pad2)
- R1 pad 2: Net-(J1-Pad3) -> /S0
- R2 pad 1: /S0 -> /S1
- R23 pad 2: Net-(R17-Pad2) -> Net-(R23-Pad2)
- R3 pad 1: /S1 -> /S2
- R4 pad 1: /S2 -> /S3
- R5 pad 1: /S3 -> /S4
- R6 pad 1: /S4 -> /S5
- R7 pad 1: /S5 -> /S6
- RV1 pad 1: +12V -> Net-(R23-Pad2)
- RV1 pad 3: Net-(R17-Pad2) -> +12V
Routing:
- net +24V: track 0.00 -> 111.8 mm, vias 0 -> 2
- net +12V: track 0.00 -> 78.6 mm, vias 0 -> 2
- net Net-(J2-Pad2): track 0.00 -> 35.0 mm
- net Net-(J2-Pad1): track 0.00 -> 29.4 mm, vias 0 -> 2
- net Net-(J2-Pad3): track 0.00 -> 28.9 mm
- net Net-(R13-Pad2): track 0.00 -> 28.7 mm, vias 0 -> 2
- net Net-(J2-Pad4): track 0.00 -> 27.9 mm
- net Net-(J2-Pad5): track 0.00 -> 26.5 mm
- net Net-(JP1-Pad2): track 0.00 -> 25.4 mm, vias 0 -> 2
- net Net-(J2-Pad6): track 0.00 -> 24.6 mm
- net Net-(R11-Pad2): track 0.00 -> 23.7 mm, vias 0 -> 2
- net Net-(D6-Pad2): track 0.00 -> 22.7 mm, vias 0 -> 2
- net Net-(C6-Pad1): track 0.00 -> 19.9 mm
- net Net-(R12-Pad2): track 0.00 -> 17.7 mm
- net Net-(D1-Pad1): track 0.00 -> 16.6 mm
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- added copper zone on B.Cu, net GND
Other:
- board outline added: 59 x 46 mm
- board text added: "+24V"
- board text added: "1"
- board text added: "10"
- board text added: "2"
- board text added: "3"
- board text added: "4"
- board text added: "5"
- board text added: "6"
- board text added: "7"
- board text added: "8"
- board text added: "9"
- board text added: "COM"
- board text added: "GND"
- board text added: "NC"
- board text added: "NO"
- board text added: "S0"
- board text added: "S1"
- board text added: "S2"
- board text added: "S3"
- board text added: "S4"
- board text added: "S5"
- board text added: "S6"
